File: PCB Design/PCB ESP32.sch (KiCad schematic (older format))
At the start: 16 parts, among them J3 GameBoy_LinkPort, J4 5vBatteryPins, J5 HV_pins, J6 LV_pins, SW1 SW_Push, U1 ESP32_DEVBOARD_WROOM, U2 SD_Card_module, U3 OledDisplay_SSD1305_128_32, U4 MicroSD_Card_module

Commit message: Change to EasyEDA
Parts:
- removed D1: StatusLED, LED_THT:LED_D5.0mm, symbol Device:LED
- removed D2: PowerLED, LED_THT:LED_D5.0mm, symbol Device:LED
- removed R1: 1k Resistor, Resistor_THT:R_Axial_DIN0207_L6.3mm_D2.5mm_P10.16mm_Horizontal, symbol Device:R
- removed R3: 10k Resistor, Resistor_THT:R_Axial_DIN0207_L6.3mm_D2.5mm_P10.16mm_Horizontal, symbol Device:R
- added D1: LED_RGBC, symbol Device:LED_RGBC
- added J1: GameBoy_LinkPort, Gekkio_Connector:GameBoy_LinkPort_DMG_Horizontal, symbol Gekkio_Connector_Specialized:GameBoy_LinkPort
- added R1, R6: 220ohm, Resistor_THT:R_Axial_DIN0207_L6.3mm_D2.5mm_P10.16mm_Horizontal, symbol pspice:R
- added R3: 10k, Resistor_THT:R_Axial_DIN0207_L6.3mm_D2.5mm_P10.16mm_Horizontal, symbol pspice:R
- J4: value 5vBatteryPins -> BatteryPins
- R2: value 1k Resistor -> 220ohm
Connections:
- wire segments 140 -> 143
Other:
- moved on the sheet: J3, J4, J5, J6, R4, R5, SW1
